File: PCB_Oximetro.kicad_pcb (KiCad board)
At the start: 2 copper layers, 61.2 x 57.9 mm, 14 parts, among them J1 Conn_01x05, J2 Conn_01x08, J3 USB_B_Micro, SW1 SW_Push, U3 LM1117MP-3.3, U5 ESP32-DEVKIT-V1

Commit message: BLK Pin update
Changed BLK pin to make the PCB 1 only front layer
Routing:
- net BLK: track 61.3 -> 2.44 mm
- net DC: track 56.1 -> 0.00 mm
- net INT: track 18.5 -> 0.00 mm
Changed lines of the file:
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@@
   (segment (start 113.06 91.3) (end 114.71 89.65) (width 0.381) (layer "F.Cu") (net 6))
   (segment (start 114.71 89.65) (end 117.1575 89.65) (width 0.381) (layer "F.Cu") (net 6))
-  (segment (start 96.71 84.58) (end 96.71 89.88) (width 0.381) (layer "B.Cu") (net 7))
-  (segment (start 99.3705 92.5405) (end 114.3595 92.5405) (width 0.381) (layer "B.Cu") (net 7))
-  (segment (start 104.995 82.255) (end 104.03 83.22) (width 0.381) (layer "B.Cu") (net 7))
-  (segment (start 96.71 89.88) (end 99.3705 92.5405) (width 0.381) (layer "B.Cu") (net 7))
-  (segment (start 104.995 61.1725) (end 104.995 82.255) (width 0.381) (layer "B.Cu") (net 7))
-  (segment (start 114.3595 92.5405) (end 115.6 91.3) (width 0.381) (layer "B.Cu") (net 7))
-  (segment (start 98.07 83.22) (end 96.71 84.58) (width 0.381) (layer "B.Cu") (net 7))
-  (segment (start 104.03 83.22) (end 98.07 83.22) (width 0.381) (layer "B.Cu") (net 7))
   (segment (start 122.775 86.665) (end 122.775 86.5725) (width 0.381) (layer "F.Cu") (net 8))
   (segment (start 118.14 91.2075) (end 118.14 91.3) (width 0.25) (layer "F.Cu") (net 8))
   (segment (start 118.14 91.3) (end 122.775 86.665) (width 0.381) (layer "F.Cu") (net 8))
   (segment (start 118.14 91.3) (end 118.7 91.3) (width 0.381) (layer "F.Cu") (net 8))
-  (segment (start 96.0905 90.7) (end 99.6 94.2095) (width 0.381) (layer "B.Cu") (net 9))
   (segment (start 97.818092 63.9) (end 96.0905 65.627592) (width 0.381) (layer "B.Cu") (net 9))
-  (segment (start 96.0905 65.627592) (end 96.0905 90.7) (width 0.381) (layer "B.Cu") (net 9))
-  (segment (start 102.455 62.445) (end 101 63.9) (width 0.381) (layer "B.Cu") (net 9))
-  (segment (start 99.6 94.2095) (end 117.7705 94.2095) (width 0.381) (layer "B.Cu") (net 9))
-  (segment (start 102.455 61.1725) (end 102.455 62.445) (width 0.381) (layer "B.Cu") (net 9))
-  (segment (start 101 63.9) (end 97.818092 63.9) (width 0.381) (layer "B.Cu") (net 9))
-  (segment (start 117.7705 94.2095) (end 120.68 91.3) (width 0.381) (layer "B.Cu") (net 9))
   (segment (start 134.92 103.2) (end 134.92 88.5575) (width 0.381) (layer "F.Cu") (net 10))
   (segment (start 134.92 88.5575) (end 132.935 86.5725) (width 0.381) (layer "F.Cu") (net 10))
   (segment (start 132.38 91.0975) (end 127.855 86.5725) (width 0.381) (layer "F.Cu") (net 11))
   (segment (start 132.38 103.2) (end 132.38 91.0975) (width 0.381) (layer "F.Cu") (net 11))
-  (segment (start 125.315 86.5725) (end 125.315 98.675) (width 0.381) (layer "F.Cu") (net 12))
-  (segment (start 125.315 98.675) (end 129.84 103.2) (width 0.381) (layer "F.Cu") (net 12))
   (segment (start 135.8875 71.8) (end 136.901 71.8) (width 0.381) (layer "F.Cu") (net 13))
   (segment (start 135.8875 71.8) (end 135.95 71.7375) (width 0.381) (layer "F.Cu") (net 13))

Commit message: Gerbers file
Generated gerbers files and drill
Connections:
- J2 pad 6: DC -> unconnected-(J2-Pin_6-Pad6)
- U5 pad 14: DC -> unconnected-(U5-D22-Pad14)
- U5 pad 15: BLK -> unconnected-(U5-D23-Pad15)
- U5 pad 25: INT -> BLK
Routing:
- net BLK: track 2.44 -> 6.65 mm

Commit message: Update PCB
Connections:
- J2 pad 6: unconnected-(J2-Pin_6-Pad6) -> DC
- U5 pad 14: unconnected-(U5-D22-Pad14) -> DC
Changed lines of the file:
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@@
     (pcbplotparams
       (layerselection 0x0001000_7fffffff)
-      (plot_on_all_layers_selection 0x0000000_00000001)
+      (plot_on_all_layers_selection 0x0001000_00000001)
       (disableapertmacros false)
       (usegerberextensions false)
@@
       (dxfimperialunits true)
       (dxfusepcbnewfont true)
-      (psnegative false)
+      (psnegative true)
       (psa4output false)
       (plotreference true)
@@
       (sketchpadsonfab false)
       (subtractmaskfromsilk false)
-      (outputformat 1)
+      (outputformat 4)
       (mirror false)
-      (drillshape 0)
+      (drillshape 2)
       (scaleselection 1)
       (outputdirectory "")
@@
   (net 33 "unconnected-(J3-ID-Pad4)")
   (net 34 "unconnected-(U5-D34-Pad19)")
-  (net 35 "unconnected-(J2-Pin_6-Pad6)")
-  (net 36 "unconnected-(U5-D22-Pad14)")
-  (net 37 "unconnected-(U5-D23-Pad15)")
+  (net 35 "DC")
+  (net 36 "unconnected-(U5-D23-Pad15)")
   (footprint "Capacitor_THT:CP_Radial_D5.0mm_P2.50mm" (layer "F.Cu")
     (at 135.95 67.05)
@@
       (net 6 "RESET") (pinfunction "Pin_5") (pintype "passive"))
     (pad "6" thru_hole oval (at 0 12.7 90) (size 1.7 1.7) (drill 1) (layers "*.Cu" "*.Mask")
-      (net 35 "unconnected-(J2-Pin_6-Pad6)") (pinfunction "Pin_6") (pintype "passive+no_connect"))
+      (net 35 "DC") (pinfunction "Pin_6") (pintype "passive"))
     (pad "7" thru_hole oval (at 0 15.24 90) (size 1.7 1.7) (drill 1) (layers "*.Cu" "*.Mask")
       (net 7 "CS") (pinfunction "Pin_7") (pintype "passive"))
@@
       (net 17 "unconnected-(U5-TX0-Pad13)") (pinfunction "TX0") (pintype "output+no_connect") (solder_mask_margin 0.102))
     (pad "14" thru_hole circle (at -12.7 17.505 270) (size 2 2) (drill 1.02) (layers "*.Cu" "*.Mask")
-      (net 36 "unconnected-(U5-D22-Pad14)") (pinfunction "D22") (pintype "bidirectional+no_connect") (solder_mask_margin 0.102))
+      (net 35 "DC") (pinfunction "D22") (pintype "bidirectional") (solder_mask_margin 0.102))
     (pad "15" thru_hole circle (at -12.7 20.045 270) (size 2 2) (drill 1.02) (layers "*.Cu" "*.Mask")
-      (net 37 "unconnected-(U5-D23-Pad15)") (pinfunction "D23") (pintype "bidirectional+no_connect") (solder_mask_margin 0.102))
+      (net 36 "unconnected-(U5-D23-Pad15)") (pinfunction "D23") (pintype "bidirectional+no_connect") (solder_mask_margin 0.102))
     (pad "16" thru_hole circle (at 12.7 20.045 270) (size 2 2) (drill 1.02) (layers "*.Cu" "*.Mask")
       (net 20 "unconnected-(U5-EN-Pad16)") (pinfunction "EN") (pintype "input+no_connect") (solder_mask_margin 0.102))
